File: Electrical/Twyst-Hardware.kicad_pcb (KiCad board)
At the start: 2 copper layers, 37 x 37 mm, 22 parts, among them J1 Conn_01x02_Pin, Q1 BSS84, SW1 SW_SPDT, U1 MCP73831-2ACI/MC, U2 AP2112K-3.3TRG1_C23380830, U4 ICM-45686, U5 BMM150, U6 ESP32-C3_SUPERMINI_TH

Commit message: Added screen module in schematics
Parts:
- added J2: Conn_01x13_Pin, Connector_PinHeader_1.00mm:PinHeader_1x13_P1.00mm_Vertical, F.Cu at (141.0, 118.5)
- added U7: ESP32-C3_SUPERMINI_TH, esp32:MODULE_ESP32-C3_SUPERMINI_TH, B.Cu at (144.0, 133.5)
