File: Electrical/Twyst-Hardware.kicad_sch (KiCad schematic)
At the start: 22 parts, among them J1 Conn_01x02_Pin, Q1 BSS84, SW1 SW_SPDT, U1 MCP73831-2ACI/MC, U2 AP2112K-3.3TRG1_C23380830, U4 ICM-45686, U5 BMM150, U6 ESP32-C3_SUPERMINI_TH

Commit message: Added screen module in schematics
Parts:
- added J2: Conn_01x13_Pin, Connector_PinHeader_1.00mm:PinHeader_1x13_P1.00mm_Vertical, symbol Connector:Conn_01x13_Pin
- added U7: ESP32-C3_SUPERMINI_TH, esp32:MODULE_ESP32-C3_SUPERMINI_TH, symbol esp32:ESP32-C3_SUPERMINI_TH
Connections:
- net +3.3V: now also J2.VCC (Pin_1), U7.3.3 (3V3)
- net GND: now also J2.GND (Pin_2), U7.G (GND)
- new net: J2.LCD_BL (Pin_9), U7.10 (GPIO10)
- new net: J2.LCD_CS (Pin_6), U7.3 (GPIO3)
- new net: J2.LCD_DC (Pin_7), U7.2 (GPIO2)
- new net: J2.LCD_RST (Pin_8), U7.1 (GPIO1)
- new net: J2.MISO (Pin_3), U7.5 (GPIO5)
- new net: J2.MOSI (Pin_4), U7.6 (GPIO6)
- new net: J2.SCLK (Pin_5), U7.4 (GPIO4)
- new net: J2.TP_INT (Pin_12), U7.21 (GPIO21)
- new net: J2.TP_RST (Pin_13), U7.20 (GPIO20)
- new net: J2.TP_SCL (Pin_11), U7.9 (GPIO9)
- new net: J2.TP_SDA (Pin_10), U7.8 (GPIO8)
- no-connect marks 28 -> 31
Other:
- note added: "Main Circuit"
- note added: "Round LCD Circuit"
